Commit message: created a new joint and a new link

File: lab3PD/urdf/dobot.urdf.xacro (robot description, xacro)
@@ -29,20 +29,38 @@
             </geometry>
             <origin xyz="0 0 0.025 " rpy="0 0 0" />
+            <material name="grey"/>
+        </visual>
+    </link>
+    <joint name="base_link1_joint" type="revolute">
+        <parent link="base"/>
+        <child link="link1"/>
+        <axis xyz="0 0 1"/>
+        <limit effort="1000.0" lower="-1.5708" upper="1.5708" velocity="0.889"/>
+        <origin xyz="0 0 0.05 " rpy="0 0 0 "/>
+    </joint>
+    <link name="link1">
+        <visual>
+            <geometry>
+                <cylinder radius="0.015" length="0.088"/>
+            </geometry>
+            <origin xyz="0 0 0.044" rpy="0 0 0" />
+            <material name="orange"/>
+        </visual>
+    </link>
+    <joint name="link1_link2_joint" type="revolute">
+        <parent link="link1"/>
+        <child link="link2"/>
+        <axis xyz="1 0 0"/>
+        <limit effort="1000.0" lower="-1.3962" upper="0" velocity="0.889"/>
+        <origin xyz="0 0 0.088" rpy="1.57 0 0 "/>
+    </joint>
+    <link name="link2">
+        <visual>
+            <geometry>
+                <cylinder radius="0.015" length="0.135"/>
+            </geometry>
+            <origin xyz="0 0 0.0675" rpy="0 0 0" />
             <material name="blue"/>
         </visual>
     </link>
-    <link name="link1">
-        <visual>
-            <geometry>
-                <cylinder radius="0.1" length="0.088"/>
-            </geometry>
-            <origin xyz="0 0 0.25" rpy="0 0 0" />
-            <material name="orange"/>
-        </visual>
-    </link>
-    <joint name="base_link_joint" type="fixed">
-        <parent link="base"/>
-        <child link="link1"/>
-        <origin xyz="0 0 0.2 " rpy="0 0 0 "/>
-    </joint>
 </robot>

Commit message: created a new dobot model with working joints basing on the tutorial examples

File: lab3PD/urdf/dobot.urdf.xacro (robot description, xacro)
@@ -1,5 +1,5 @@
 <?xml version="1.0"?>
 <robot xmlns:xacro="http://www.ros.org/wiki/xacro" name="dobot">
-    <xacro:property name="values_file" value="$(find lab3PD)/values.yaml"/>
+    <xacro:property name="values_file" value="$(find lab3PD)/urdf/values.yaml"/>
     <xacro:property name="params" value="${xacro.load_yaml(values_file)}"/>
     <xacro:property name="l0" value="${params['link']['l0']}"/>
