Commit message: added a sphere to the "knee" of the dobot

File: urdf_tutorial/urdf/dobot.urdf.xacro (robot description, xacro)
@@ -42,8 +42,8 @@
       <visual>
         <geometry>
-          <box size="0.003 ${width-0.01} ${l0_height - 0.01}"/>
+          <box size="${l0_height - 0.02} ${width-0.01} 0.003"/>
         </geometry>
         <material name = "white"/>
-        <origin rpy="0 0 0" xyz="${width/2} 0 ${l0_height / 2}"/>
+        <origin rpy="0 0 0" xyz="${width/2 - (l0_height - 0.01)/2} 0 ${l0_height}"/>
       </visual>
   </link>
@@ -72,5 +72,5 @@
       <visual>
         <geometry>
-          <cylinder length="${l2_length + 0.04}" radius="0.02"/>
+          <cylinder length="${l2_length + 0.02}" radius="0.02"/>
         </geometry>
         <origin xyz="0 0 ${l2_length/2}" rpy="0 0 0"/>
@@ -87,5 +87,14 @@
       </visual>
   </link>
-  <joint name="arm_2_joint" type="revolute">
+  <link name="arm_joint_sphere">
+    <visual>
+        <geometry>
+            <sphere radius="0.03"/>
+        </geometry>
+        <origin xyz="0 0 0" rpy="0 0 0"/>
+        <material name="blue"/>
+    </visual>
+  </link>
+  <joint name="arm_rotbase_joint" type="revolute">
     <axis xyz="0 1 0"/>
     <limit effort="1000.0" lower="${j1_min}" upper="${j1_max}" velocity="0.5"/>
@@ -94,9 +103,14 @@
     <origin xyz="0 0 ${l1_height}"/>
   </joint>
-  <joint name="arm_3_joint" type="revolute">
+  <joint name="arm_arm_joint" type="revolute">
     <axis xyz="0 1 0"/>
     <limit effort="1000.0" lower="${j2_min}" upper="${j2_max}" velocity="0.5"/>
     <parent link="lower_arm"/>
     <child link="upper_arm"/>
+    <origin xyz="0 0 ${l2_length}"/>
+  </joint>
+  <joint name="sphere_joint" type="fixed">
+    <parent link="lower_arm"/>
+    <child link="arm_joint_sphere"/>
     <origin xyz="0 0 ${l2_length}"/>
   </joint>

Commit message: addded the power button

File: urdf_tutorial/urdf/dobot.urdf.xacro (robot description, xacro)
@@ -29,4 +29,7 @@
     <color rgba="0.03 0 0.8 1"/>
 </material>
+<material name="red">
+    <color rgba="1 0 0 1"/>
+</material>
   <xacro:property name="width" value="0.18" />
   <link name="base">
@@ -51,4 +54,18 @@
     <parent link="base"/>
     <child link="front_label"/>
+    <origin xyz="0 0 0"/>
+  </joint>\
+  <link name="power_button">
+      <visual>
+        <geometry>
+          <cylinder length="0.003" radius="0.01"/>
+        </geometry>
+        <material name = "red"/>
+        <origin rpy="0 0 0" xyz="${-width/2 + (l0_height - 0.01)/2} ${width/2-0.02} ${l0_height}"/>
+      </visual>
+  </link>
+  <joint name="power_joint" type="fixed">
+    <parent link="base"/>
+    <child link="power_button"/>
     <origin xyz="0 0 0"/>
   </joint>

Commit message: working ForwardKin

File: urdf_tutorial/urdf/dobot.urdf.xacro (robot description, xacro)
@@ -1,5 +1,5 @@
 <?xml version="1.0"?>
 <robot name="macroedsad" xmlns:xacro="http://ros.org/wiki/xacro">
-  <xacro:property name="params" value="${xacro.load_yaml('/home/antek/anro_ws/src/urdf_tutorial/parameters/size_values.yaml')}"/>
+  <xacro:property name="params" value="${xacro.load_yaml('$(find urdf_tutorial)/parameters/size_values.yaml')}"/>
   <xacro:property name="l0_height" value="${params['links_sizes']['link0']}" />
   <xacro:property name="l1_height" value="${params['links_sizes']['link1']}" />
@@ -167,5 +167,5 @@
       <visual>
         <geometry>
-          <box size="0.02 0.02 0.03"/>
+          <box size="0.02 0.02 0.04"/>
         </geometry>
         <material name = "blue"/>
@@ -176,5 +176,5 @@
     <parent link="effector_rot_base"/>
     <child link="gripper"/>
-    <origin xyz="0 0 -0.015"/>
+    <origin xyz="0 0 -0.02"/>
   </joint>
 </robot>

Commit message: changed launch and moved kinematics down a bit

File: urdf_tutorial/urdf/dobot.urdf.xacro (robot description, xacro)
@@ -167,5 +167,5 @@
       <visual>
         <geometry>
-          <box size="0.02 0.02 0.04"/>
+          <box size="0.015 0.028 0.04"/>
         </geometry>
         <material name = "blue"/>
@@ -178,3 +178,17 @@
     <origin xyz="0 0 -0.02"/>
   </joint>
+  <link name="actuator">
+      <visual>
+        <geometry>
+          <box size="0.015 0.025 0.02"/>
+        </geometry>
+        <material name = "red"/>
+        <origin rpy="0 0 0" xyz="0 0.0125 0"/>
+      </visual>
+  </link>
+  <joint name="actuator_joint" type="fixed">
+    <parent link="gripper"/>
+    <child link="actuator"/>
+    <origin xyz="0 0.016 0"/>
+  </joint>
 </robot>

Commit message: lab6PD first stage

File: urdf_tutorial/urdf/dobot.urdf.xacro (robot description, xacro)
@@ -7,4 +7,5 @@
   <xacro:property name="l3_length" value="${params['links_sizes']['link3']}"/>
   <xacro:property name="l4_length" value="${params['links_sizes']['link4']}"/>
+  <xacro:property name="camera_distance" value="${params['links_sizes']['camera_link']}"/>
   <xacro:property name="j0_min" value="${params['joints_limits']['joint0']['min']}" />
   <xacro:property name="j0_max" value="${params['joints_limits']['joint0']['max']}" />
@@ -95,4 +96,34 @@
       </visual>
   </link>
+  <link name="camera_link">
+      <visual>
+        <geometry>
+          <box size="${camera_distance/4} 0.012 0.012"/>
+        </geometry>
+        <material name = "blue"/>
+        <origin rpy="0 0 0" xyz="${camera_distance/8} 0 0"/>
+      </visual>
+  </link>
+  <link name="camera">
+      <visual>
+        <geometry>
+          <box size="0.025 0.09 0.025"/>
+        </geometry>
+        <material name = "red"/>
+        <origin rpy="0 0 0" xyz="0 0 0"/>
+      </visual>
+  </link>
+  <joint name="camera_joint" type="fixed">
+    <axis xyz="0 1 0"/>
+    <parent link="effector"/>
+    <child link="camera_link"/>
+    <origin xyz="${l4_length - 0.02} 0 0"/>
+  </joint>
+  <joint name="camera_joint2" type="fixed">
+    <axis xyz="0 1 0"/>
+    <parent link="camera_link"/>
+    <child link="camera"/>
+    <origin rpy="3.1415 0 0" xyz="${camera_distance/4} 0 0"/>
+  </joint>
   <link name="upper_arm">
       <visual>
